Commit message: fine tunning to xacro model

File: urdf/gocator_3109.urdf.xacro (robot description, xacro)
@@ -25,8 +25,9 @@
             </collision>
         </link>
+        <!-- TODO: Grow a cylinder to Y>0 to model the conector (radius 1cm, length 4cm) -->
         <joint name="${name}_point_cloud_anchor" type="fixed" >
             <parent link="${name}"/>
             <child link="${name}_point_cloud"/>
-            <origin xyz="0 0 ${0.095+0.157+0.035}" rpy="0 3.141592 0"/>
+            <origin xyz="0 0 ${0.0942+0.157+0.035}" rpy="0 3.141592 0"/>  <!--27.9cm from parent -->
         </joint>
         <link name="${name}_point_cloud"/>

Commit message: Fixed Time stamp bug on point cloud publisher and urdf bug on gocator_point_cloud frame

File: urdf/gocator_3109.urdf.xacro (robot description, xacro)
@@ -29,5 +29,5 @@
             <parent link="${name}"/>
             <child link="${name}_point_cloud"/>
-            <origin xyz="0 0 ${0.0942+0.157+0.035}" rpy="0 3.141592 0"/>  <!--27.9cm from parent -->
+            <origin xyz="0 0 ${0.0942+0.157+0.035}" rpy="0 3.141592 1.570796"/>  <!--27.9cm from parent -->
         </joint>
         <link name="${name}_point_cloud"/>

Commit message: Fixed on gocator_point_cloud frame yaw angle

File: urdf/gocator_3109.urdf.xacro (robot description, xacro)
@@ -29,5 +29,5 @@
             <parent link="${name}"/>
             <child link="${name}_point_cloud"/>
-            <origin xyz="0 0 ${0.0942+0.157+0.035}" rpy="0 3.141592 1.570796"/>  <!--27.9cm from parent -->
+            <origin xyz="0 0 ${0.0942+0.157+0.035}" rpy="0 3.141592 -1.570796"/>  <!--27.9cm from parent -->
         </joint>
         <link name="${name}_point_cloud"/>

Commit message: Added mesh file for a more realistic visualization model of gocator

File: urdf/gocator_3109.urdf.xacro (robot description, xacro)
@@ -14,5 +14,6 @@
                 <origin xyz="0 0 0.05" rpy="0 0 0"/>
                 <geometry>
-                    <box size="0.156 0.05 0.1"/>
+                    <!-- <box size="0.156 0.05 0.1"/> -->
+                    <mesh filename="package://gocator_3100/urdf/gocator_3109a.stl"/>
                 </geometry>
                 <material name="Gocator/Black"/>

Commit message: Scaling gocator mesh to meters

File: urdf/gocator_3109.urdf.xacro (robot description, xacro)
@@ -15,5 +15,5 @@
                 <geometry>
                     <!-- <box size="0.156 0.05 0.1"/> -->
-                    <mesh filename="package://gocator_3100/urdf/gocator_3109a.stl"/>
+                    <mesh filename="package://gocator_3100/urdf/gocator_3109a.stl" scale="0.001 0.001 0.001"/>
                 </geometry>
                 <material name="Gocator/Black"/>

Commit message: Removing offset at urdf for visual mounting point

File: urdf/gocator_3109.urdf.xacro (robot description, xacro)
@@ -12,5 +12,6 @@
         <link name="${name}">
             <visual>
-                <origin xyz="0 0 0.05" rpy="0 0 0"/>
+                <!-- <origin xyz="0 0 0.05" rpy="0 0 0"/> -->
+                <origin xyz="0 0 0" rpy="0 0 0"/> -->
                 <geometry>
                     <!-- <box size="0.156 0.05 0.1"/> -->

Commit message: Fixed typo in gocator_3109.urdf.xacro

File: urdf/gocator_3109.urdf.xacro (robot description, xacro)
@@ -13,5 +13,5 @@
             <visual>
                 <!-- <origin xyz="0 0 0.05" rpy="0 0 0"/> -->
-                <origin xyz="0 0 0" rpy="0 0 0"/> -->
+                <origin xyz="0 0 0" rpy="0 0 0"/>
                 <geometry>
                     <!-- <box size="0.156 0.05 0.1"/> -->
