Commit message: Increases the collision geometry, the last one was too small

File: urdf/gocator_3110.urdf.xacro (robot description, xacro)
@@ -21,7 +21,7 @@
             </visual>
             <collision>
-                <origin xyz="0 0 0.04" rpy="0 0 0"/>
+                <origin xyz="0 0 0.05" rpy="0 0 0"/>
                 <geometry>
-                    <box size="0.300 0.04 0.08"/>
+                    <box size="0.310 0.10 0.1"/>
                 </geometry>
             </collision>
